Commit message: Implement robot.R_tool and robot.p_tool to allow for arbitrary tool transform. Supported in fwdkin, robotjacobian, robot6_sphericalwrist_invkin, and urdf loader.

File: test/irb6640_180_255_nogeom_twist.urdf (robot description, URDF)
Before this commit: robot abb_irb6640_180_255, 10 links, 9 joints
Joints:
- joint joint_6-tool0: origin xyz=0 0 0 rpy=0 1.57079632679 0 -> xyz=0 0 0 rpy=3.14159265358 0 1.57079632679

File: test/sda10f_nogeom.urdf (robot description, URDF)
Before this commit: robot motoman_sda10f, 19 links, 18 joints
Joints:
- joint arm_left_joint_1_s: origin xyz=0.09996 0.0275 0.32214 rpy=1.57 0 0.0 -> xyz=0.09996 0.0275 0.32214 rpy=1.57079632679 0 0.0
- joint arm_left_joint_2_l: origin xyz=0 0.0577 -0.2255 rpy=-1.57 0 0 -> xyz=0 0.0577 -0.2255 rpy=-1.57079632679 0 0
- joint arm_left_joint_3_e: origin xyz=0 0.1690 -0.0454 rpy=1.57 0 0 -> xyz=0 0.1690 -0.0454 rpy=1.57079632679 0 0
- joint arm_left_joint_4_u: origin xyz=0 -0.0085 -0.181 rpy=-1.57 0 0 -> xyz=0 -0.0085 -0.181 rpy=-1.57079632679 0 0
- joint arm_left_joint_5_r: origin xyz=0 0.1936 0.0155 rpy=1.57 0 0 -> xyz=0 0.1936 0.0155 rpy=1.57079632679 0 0
- joint arm_left_joint_6_b: origin xyz=0 0.0080 -0.155 rpy=-1.57 0 0 -> xyz=0 0.0080 -0.155 rpy=-1.57079632679 0 0
- joint arm_left_joint_7_t: origin xyz=0 0.168 -0.015 rpy=1.57 0 0 -> xyz=0 0.168 -0.015 rpy=1.57079632679 0 0
- joint arm_left_joint_tool0: origin xyz=0 0 0.0 rpy=0 0 -3.13 -> xyz=0 0 0.0 rpy=0 0 -3.14159265358
- joint arm_right_joint_1_s: origin xyz=0.09996 -0.0275 0.32214 rpy=1.57 0 -3.14 -> xyz=0.09996 -0.0275 0.32214 rpy=1.57079632679 0 -3.14159265358
- joint arm_right_joint_2_l: origin xyz=0 0.0577 -0.2255 rpy=-1.57 0 0 -> xyz=0 0.0577 -0.2255 rpy=-1.57079632679 0 0
- joint arm_right_joint_3_e: origin xyz=0 0.1690 -0.0454 rpy=1.57 0 0 -> xyz=0 0.1690 -0.0454 rpy=1.57079632679 0 0
- joint arm_right_joint_4_u: origin xyz=0 -0.0085 -0.181 rpy=-1.57 0 0 -> xyz=0 -0.0085 -0.181 rpy=-1.57079632679 0 0
- joint arm_right_joint_5_r: origin xyz=0 0.1936 0.0155 rpy=1.57 0 0 -> xyz=0 0.1936 0.0155 rpy=1.57079632679 0 0
- joint arm_right_joint_6_b: origin xyz=0 0.0080 -0.155 rpy=-1.57 0 0 -> xyz=0 0.0080 -0.155 rpy=-1.57079632679 0 0
- joint arm_right_joint_7_t: origin xyz=0 0.168 -0.015 rpy=1.57 0 0 -> xyz=0 0.168 -0.015 rpy=1.57079632679 0 0
- joint arm_right_joint_tool0: origin xyz=0 0 0.0 rpy=0 0 -3.13 -> xyz=0 0 0.0 rpy=0 0 -3.14159265358
